Commit message: Split mirobot into shaft + vacuum gripper

File: data/robots/mirobot_vacuum.urdf (robot description, URDF)
Before this commit: robot mirobot, 8 links, 7 joints
Links:
- added link Vacuum, mass 0.001; collision mesh filename=mirobot/Vacuum.STL; visual mesh filename=mirobot/Vacuum.STL
Joints:
- added joint VacuumJoint: type fixed, parent Link6, child Vacuum, origin xyz=0 0 0 rpy=0 0 0
